Commit message: Added lidar sensor to URDF

File: shanti_base/src/description/shanti_description.urdf (robot description, URDF)
Before this commit: robot sam_bot, 4 links, 3 joints
Links:
- added link lidar_link; collision cylinder length=${lidar_width} radius=${lidar_radius}; visual cylinder length=${lidar_width} radius=${lidar_radius}
Joints:
- added joint lidar_joint: type fixed, parent base_link, child lidar_link, origin xyz=0 0 0.111
