Commit message: got the xoff set to the right value

File: shanti_base/src/description/shanti_6w_description.urdf (robot description, URDF)
Before this commit: robot shanti, 6 links, 5 joints
Links:
- link base_link: geometry visual box size=${base_length} ${base_width} ${base_height}

File: shanti_base/src/description/shanti_description.xacro (robot description, xacro)
@@ -1,4 +1,4 @@
 <?xml version="1.0"?>
-<robot name="shanti" xmlns:xacro="http://ros.org/wiki/xacro">
+<robot name="shanti" xmlns:xacro="http://www.ros.org/wiki/xacro">
   <!-- Define robot constants in meters-->
   <xacro:property name="base_width" value="0.31" />
@@ -95,5 +95,5 @@
     <visual>
       <geometry>
-        <sphere radius="${(wheel_radius+wheel_zoff-(base_height/2))}" />
+        <sphere radius="${wheel_radius+wheel_zoff-(base_height/2)}" />
       </geometry>
       <material name="Cyan">
@@ -104,8 +104,8 @@
       <origin xyz="0 0 0" rpy="0 0 0" />
       <geometry>
-        <sphere radius="${(wheel_radius+wheel_zoff-(base_height/2))}" />
+        <sphere radius="${wheel_radius+wheel_zoff-(base_height/2)}" />
       </geometry>
     </collision>
-    <xacro:sphere_inertia m="0.5" r="${(wheel_radius+wheel_zoff-(base_height/2))}" />
+    <xacro:sphere_inertia m="0.5" r="${wheel_radius+wheel_zoff-(base_height/2)}" />
   </link>
   <joint name="caster_joint" type="fixed">
