Commit message: Fixed some files for GPS display

File: shanti_base/description/shanti_description.urdf (robot description, URDF)
Before this commit: robot sam_bot, 5 links, 4 joints
Links:
- added link gps_link
Joints:
- added joint gps_joint: type fixed, parent base_link, child gps_link, origin xyz=0 0 0 rpy=0 0 0
