Commit message: This is a .xacro file, not a .urdf file

File: shanti_base/description/shanti_6w_description.xacro (robot description, xacro)
@@ -1,4 +1,4 @@
 <?xml version="1.0"?>
-<robot name="shanti" xmlns:xacro="http://ros.org/wiki/xacro">
+<robot name="shanti" xmlns:xacro="http://www.ros.org/wiki/xacro">
   <!-- Define robot constants in meters-->
   <xacro:property name="base_width" value="0.6604" />
@@ -29,5 +29,5 @@
         iyz="0" izz="${(m/2) * (r*r)}" />
     </inertial>
-  </xacro:macro>0,292
+  </xacro:macro>
   <xacro:macro name="sphere_inertia" params="m r">
     <inertial>
@@ -90,5 +90,5 @@
   <xacro:wheel prefix="drivewhl_r2" x_reflect="0" y_reflect="-1" />
   <xacro:wheel prefix="drivewhl_r3" x_reflect="1" y_reflect="-1" />
-  <!-- Caster Wheel
+  <!-- Caster Wheel  -->
   <link name="front_caster">
     <visual>
@@ -113,5 +113,4 @@
     <origin xyz="${caster_xoff} 0.0 ${-(base_height/2)}" rpy="0 0 0" />
   </joint>
--->
   <!-- IMU Sensor -->
   <link name="imu_link">
