Commit message: fixed the mass issue the made the robot fly...

File: shanti_base/description/shanti_6w_description.urdf (robot description, URDF)
Before this commit: robot shanti, 6 links, 5 joints
Links:
- removed link front_caster
Joints:
- removed joint caster_joint

Commit message: Restoring Navigation files

File: shanti_base/description/shanti_6w_description.urdf (robot description, URDF)
Before this commit: robot shanti, 12 links, 11 joints
Links:
- removed link drivewhl_l1_link
- removed link drivewhl_l2_link
- removed link drivewhl_l3_link
- removed link drivewhl_r1_link
- removed link drivewhl_r2_link
- removed link drivewhl_r3_link
- link base_link: mass 0.1 -> None; geometry visual box size=${base_length} ${base_width} ${base_height}
- link front_caster: mass 0.5 -> None; geometry collision sphere radius=${(wheel_radius+wheel_zoff-(base_height/2))}; visual sphere radius=${(wheel_radius+wheel_zoff-(base_height/2))}
- link imu_link: mass 0.1 -> None
- link lidar_link: mass 0.5 -> None; geometry collision cylinder length=${lidar_width} radius=${lidar_radius}; visual cylinder length=${lidar_width} radius=${lidar_radius}
Joints:
- removed joint drivewhl_l1_joint
- removed joint drivewhl_l2_joint
- removed joint drivewhl_l3_joint
- removed joint drivewhl_r1_joint
- removed joint drivewhl_r2_joint
- removed joint drivewhl_r3_joint
- joint base_joint: origin xyz=0.0 0.0 -0.40159999999999996 rpy=0 0 0 -> xyz=0.0 0.0 ${-(wheel_radius+wheel_zoff)} rpy=0 0 0
- joint caster_joint: origin xyz=0.14 0.0 -0.3175 rpy=0 0 0 -> xyz=${caster_xoff} 0.0 ${-(base_height/2)} rpy=0 0 0

File: shanti_base/description/shanti_description.urdf (robot description, URDF)
Before this commit: robot shanti, 8 links, 7 joints
Links:
- removed link drivewhl_l_link
- removed link drivewhl_r_link
- link base_link: mass 15 -> None; geometry collision box size=${base_length} ${base_width} ${base_height}; visual box size=${base_length} ${base_width} ${base_height}
- link front_caster: mass 0.5 -> None; geometry collision sphere radius=${wheel_radius+wheel_zoff-(base_height/2)}; visual sphere radius=${wheel_radius+wheel_zoff-(base_height/2)}
- link imu_link: mass 0.1 -> None
- link lidar_link: mass 0.5 -> None; geometry collision cylinder length=${lidar_width} radius=${lidar_radius}; visual cylinder length=${lidar_width} radius=${lidar_radius}
Joints:
- removed joint drivewhl_l_joint
- removed joint drivewhl_r_joint
- joint base_joint: origin xyz=0.0 0.0 -0.15000000000000002 rpy=0 0 0 -> xyz=0.0 0.0 ${-(wheel_radius+wheel_zoff)} rpy=0 0 0
- joint caster_joint: origin xyz=0.14 0.0 -0.09 rpy=0 0 0 -> xyz=${caster_xoff} 0.0 ${-(base_height/2)} rpy=0 0 0

Commit message: trying real hard here...

File: shanti_base/description/shanti_6w_description.urdf (robot description, URDF)
Before this commit: robot shanti, 5 links, 4 joints
Links:
- added link camera_front; collision cylinder length=${camera_width} radius=${camera_radius}; visual cylinder length=${camera_width} radius=${camera_radius}
- added link camera_rear; collision cylinder length=${camera_width} radius=${camera_radius}; visual cylinder length=${camera_width} radius=${camera_radius}
Joints:
- added joint camera_front_joint: type fixed, parent base_link, child camera_front, origin xyz=0 0 1.0 rpy=0 0 0
- added joint camera_rear_joint: type fixed, parent base_link, child camera_rear, origin xyz=0 0 1.0 rpy=0 0 3.14159
