Commit message: Fixed tfs, working on costmaps

File: shanti_base/description/shanti_6w_lidar_description.urdf (robot description, URDF)
Before this commit: robot shanti, 6 links, 5 joints
Links:
- link base_footprint: geometry collision box size=${base_length} ${base_width} ${base_height}; visual box size=${base_length} ${base_width} ${base_height}
- link base_link: geometry 
Joints:
- joint base_joint: origin xyz=0.0 0.0 ${-(wheel_radius+wheel_zoff)} rpy=0 0 0 -> xyz=0.0 0.0 ${(wheel_radius+wheel_zoff)} rpy=0 0 0
- joint gps_joint: parent base_link -> base_footprint
- joint imu_joint: parent base_link -> base_footprint
- joint lidar_back_right_joint: parent base_link -> base_footprint
- joint lidar_front_left_joint: parent base_link -> base_footprint

Commit message: Added a camera to the urdf file ... it is high up at the center of the robot.  When you run rviz you can add a camera sensor by topic.../camera_sensor/image_raw/Camera. and you will see the image from that camera.  You can then use that image topic to do further processing

File: shanti_base/description/shanti_6w_lidar_description.urdf (robot description, URDF)
Before this commit: robot shanti, 6 links, 5 joints
Links:
- added link camera_link, mass 0.1; collision box size=0.1 0.1 0.1; visual box size=0.1 0.1 0.1
Joints:
- added joint camera_joint: type fixed, parent base_footprint, child camera_link, origin xyz=0.0 0.0 0.8 rpy=0 0 0

Commit message: This  allows  the robot to go  around the whole course and also over the bridge.

File: shanti_base/description/shanti_6w_lidar_description.urdf (robot description, URDF)
Before this commit: robot shanti, 7 links, 6 joints
Joints:
- joint lidar_back_right_joint: origin xyz=-0.55 -0.4 0.2 rpy=0 3.14 0 -> xyz=-0.55 -0.4 0.5 rpy=0 3.14 0
- joint lidar_front_left_joint: origin xyz=0.55 0.4 0.2 rpy=0 3.14 0 -> xyz=0.55 0.4 0.5 rpy=0 3.14 0

Commit message: Added a camera at the 5 meters up and 3 meter ahead of the robot.  Added a simple thresholding lane extraction function (lane_segmentation_to_pointcloud.py ... The system is able to generate lane lines in point cloud format in RVIZ.  I also added these to the costmap.... need to see if it will now follow lanes.
This can be used as a placehodler for our actual lane segmentation algorithm.

File: shanti_base/description/shanti_6w_lidar_description.urdf (robot description, URDF)
Before this commit: robot shanti, 7 links, 6 joints
Joints:
- joint camera_joint: origin xyz=0.0 0.0 0.8 rpy=0 0 0 -> xyz=3.0 0.0 5.0 rpy=0 1.5707  0

Commit message: moved lane to point cloud  to perception and tested lane algorithim in sim.  It works but needs tuning.

File: shanti_base/description/shanti_6w_lidar_description.urdf (robot description, URDF)
Before this commit: robot shanti, 7 links, 6 joints
Joints:
- joint camera_joint: origin xyz=3.0 0.0 5.0 rpy=0 1.5707  0 -> xyz=2.5 0.0 4.0 rpy=0 1.5707  0
