Commit message: Added a 2 Diff wheel 1 caster robot description, and organized urdf files to be modular for easy creation of alternative robots

File: base/shanti_base/description/sensors/camera.xacro (robot description, xacro)
@@ -4,5 +4,5 @@
     <parent link="base_link"/>
     <child link ="camera_link"/>
-    <origin xyz="${base_width/2} 0 ${base_height/3}"/>
+    <origin xyz="${base_length/2} 0 ${base_height/3}"/>
   </joint>
   <link name="camera_link">

File: base/shanti_base/description/sensors/imu.xacro (robot description, xacro)
@@ -4,14 +4,16 @@
     <parent link="base_link"/>
     <child link ="imu_link"/>
-    <origin xyz="0.2 0 ${base_height/2 + imu_height / 2}"/>
+    <origin xyz="0 0 ${base_height/2 + lidar_length / 2}"/>
   </joint>
   <link name="imu_link">
-    <visual>
+    <!-- <visual>
       <geometry>
         <box size="${imu_length} ${imu_width} ${imu_height}" />
       </geometry>
       <material name="orange"/>
-    </visual>
-    <xacro:box_inertia m="0.1" w="0.1" d="0.1" h="0.1" />
+    </visual> -->
+    <!-- <xacro:inertial_box mass="0.1" x="${imu_length}" y="${imu_width}" z="${imu_height}">
+      <origin xyz="0 0 0" rpy="0 0 0"/>
+    </xacro:inertial_box> -->
   </link>
   <gazebo reference="imu_link">

File: base/shanti_base/description/sensors/lidar.xacro (robot description, xacro)
@@ -4,5 +4,5 @@
     <parent link="base_link"/>
     <child link ="lidar_link"/>
-    <origin xyz="0 0 ${base_height/2 + lidar_length}"/>
+    <origin xyz="0 0 ${base_height/2 + lidar_length/2}"/>
   </joint>
   <link name="lidar_link">
@@ -20,5 +20,5 @@
       </geometry>
     </collision>
-    <xacro:inertial_cylinder mass="0.1" length="0.05" radius="0.05">
+    <xacro:inertial_cylinder mass="0.1" length="${lidar_length}" radius="${lidar_radius}">
         <origin xyz="0 0 0" rpy="0 0 0"/>
     </xacro:inertial_cylinder>
